File: Hardware/HighBall_Hardware_v1/Avionics_Main_Board.brd (EAGLE design)
At the start: 160 x 100 mm, 7 parts

Commit message: Fixed battery connector
Connections:
- net GND: now also J-01.2; no longer J-01.1
- net VBAT: now also J-01.1; no longer J-01.2
Changed lines of the file:
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@@
 <signals>
 <signal name="VBAT">
-<contactref element="J-01" pad="2"/>
 <contactref element="VR-01" pad="IN+"/>
 <contactref element="VR-02" pad="IN+"/>
+<contactref element="J-01" pad="1"/>
+<wire x1="3.81" y1="88.7222" x2="27.94" y2="92.71" width="0" layer="19" extent="1-1"/>
 <wire x1="27.94" y1="46.99" x2="27.94" y2="92.71" width="0" layer="19" extent="1-1"/>
-<wire x1="3.81" y1="92.5778" x2="27.94" y2="46.99" width="0" layer="19" extent="1-1"/>
 </signal>
 <signal name="GND">
-<contactref element="J-01" pad="1"/>
 <contactref element="VR-01" pad="IN-"/>
 <contactref element="VR-01" pad="OUT-"/>
@@
 <contactref element="B1" pad="GND1"/>
 <contactref element="U$2" pad="GND"/>
+<contactref element="J-01" pad="2"/>
 <wire x1="11.43" y1="46.99" x2="110.49" y2="46.99" width="0" layer="19" extent="1-1"/>
 <wire x1="11.43" y1="53.34" x2="11.43" y2="46.99" width="0" layer="19" extent="1-1"/>
-<wire x1="3.81" y1="88.7222" x2="11.43" y2="53.34" width="0" layer="19" extent="1-1"/>
-<wire x1="11.43" y1="92.71" x2="3.81" y2="88.7222" width="0" layer="19" extent="1-1"/>
+<wire x1="11.43" y1="92.71" x2="11.43" y2="53.34" width="0" layer="19" extent="1-1"/>
+<wire x1="3.81" y1="92.5778" x2="11.43" y2="92.71" width="0" layer="19" extent="1-1"/>
 <wire x1="11.43" y1="7.62" x2="11.43" y2="46.99" width="0" layer="19" extent="1-1"/>
 <wire x1="-15.113" y1="-93.98" x2="11.43" y2="7.62" width="0" layer="19" extent="1-1"/>
