File: Hardware/HighBall_Hardware_v1/Avionics_Main_Board.brd (EAGLE design)
At the start: 160 x 100 mm, 16 parts

Commit message: Added RockBLOCK to schematic
Parts:
- added COMM-01: (no value), SparkFun-Connectors:1X10
- moved GPS-01 307.8 mm to (125.7, 54.6)
- moved PIT-02 271.3 mm to (99.1, 54.6)
- moved PIT-01 264.0 mm to (119.4, 52.1), turned to 180 degrees
- moved Q-01 251.4 mm to (27.9, 108.0)
- moved Q-02 247.7 mm to (27.9, 99.1)
- moved HE-02 239.1 mm to (17.8, 101.6), turned to 270 degrees
- moved HE-01 234.1 mm to (17.8, 109.2), turned to 270 degrees
- moved TIT-01 232.1 mm to (181.6, 63.5), turned to 90 degrees
- moved LC-01 218.8 mm to (105.4, 86.4), turned to 180 degrees
- moved M-01 204.3 mm to (17.8, 86.4), turned to 90 degrees
- moved M-02 195.6 mm to (17.8, 73.7), turned to 90 degrees
- moved IMU-01 175.1 mm to (130.8, -1.27), turned to 90 degrees
- moved VR-02 74.4 mm to (85.1, 102.9), turned to 0 degrees
- moved C-1 63.1 mm to (63.5, 45.7), flipped to the bottom, turned to 90 degrees
- moved VR-01 61.9 mm to (38.1, 102.9), turned to 0 degrees
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Connections:
- new net COMM-01-CTS: COMM-01.2
- new net COMM-01-NETAV: C-1.24, COMM-01.4
- new net COMM-01-ON/OFF: C-1.25, COMM-01.7
- new net COMM-01-RI: C-1.3, COMM-01.5
- new net COMM-01-RTS: COMM-01.3
- new net COMM-01-RXD: C-1.19, COMM-01.1
- new net COMM-01-TXD: C-1.18, COMM-01.6
- net GND: now also COMM-01.10
- net VCC_1: now also COMM-01.8
Other:
- board outline removed

Commit message: Setup source files for control payload
Parts:
- moved TIT-01 52.5 mm to (137.2, 91.4)
Changed lines of the file:
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@@
 <drawing>
 <settings>
-<setting alwaysvectorfont="no"/>
+<setting alwaysvectorfont="yes"/>
 <setting verticaltext="up"/>
 </settings>
@@
 <element name="VR-02" library="High Ball Library" package="RIORAND_LM2596_BREAKOUT" value="3.3V" x="85.09" y="102.87"/>
 <element name="C-1" library="SparkFun-Boards" library_urn="urn:adsk.eagle:library:509" package="ARDUINO_MEGA" package3d_urn="urn:adsk.eagle:package:37320/1" value="ARDUINO_MEGA_R3FULL" x="63.5" y="45.72" rot="MR90"/>
-<element name="TIT-01" library="High Ball Library" package="TO92" package3d_urn="urn:adsk.eagle:package:28523/2" value="LM335TO-92" x="181.61" y="63.5" rot="R90"/>
+<element name="TIT-01" library="High Ball Library" package="TO92" package3d_urn="urn:adsk.eagle:package:28523/2" value="LM335TO-92" x="137.16" y="91.44" rot="R90"/>
 <element name="IMU-01" library="High Ball Library" package="RAZOR_IMU" value="RAZOR_IMU" x="130.81" y="-1.27" rot="R90"/>
 <element name="LC-01" library="SparkFun-Boards" library_urn="urn:adsk.eagle:library:509" package="SPARKFUN_LOGIC_LEVEL_CONVERTER_LOCK" package3d_urn="urn:adsk.eagle:package:37319/1" value="SPARKFUN_LOGIC_LEVEL_CONVERTERLOCK" x="105.41" y="86.36" rot="R180"/>
@@
 <wire x1="129.54" y1="22.225" x2="161.29" y2="104.14" width="0" layer="19" extent="1-1"/>
 <wire x1="100.457" y1="85.09" x2="129.54" y2="22.225" width="0" layer="19" extent="1-1"/>
-<wire x1="181.61" y1="64.77" x2="100.457" y2="85.09" width="0" layer="19" extent="1-1"/>
-<wire x1="77.47" y1="119.38" x2="181.61" y2="64.77" width="0" layer="19" extent="1-1"/>
+<wire x1="137.16" y1="92.71" x2="100.457" y2="85.09" width="0" layer="19" extent="1-1"/>
+<wire x1="77.47" y1="119.38" x2="137.16" y2="92.71" width="0" layer="19" extent="1-1"/>
 <wire x1="39.37" y1="34.29" x2="77.47" y2="119.38" width="0" layer="19" extent="1-1"/>
 </signal>
@@
 <contactref element="C-1" pad="GND@1"/>
 <contactref element="TIT-01" pad="3"/>
-<wire x1="39.37" y1="39.37" x2="181.61" y2="62.23" width="0" layer="19" extent="1-1"/>
+<wire x1="39.37" y1="39.37" x2="137.16" y2="90.17" width="0" layer="19" extent="1-1"/>
 </signal>
 <signal name="TIT-01">
 <contactref element="C-1" pad="A2"/>
 <contactref element="TIT-01" pad="2"/>
-<wire x1="39.37" y1="52.07" x2="179.705" y2="63.5" width="0" layer="19" extent="1-1"/>
+<wire x1="39.37" y1="52.07" x2="135.255" y2="91.44" width="0" layer="19" extent="1-1"/>
 </signal>
 <signal name="IMU-01-RX">
